File: EagleAirPoll/SchemaFin.brd (EAGLE design)
At the start: 99.1 x 99.1 mm, 5 parts

Commit message: Remove consistency errors
Parts:
- renumbered JP1 to SDS011, JP2 to DHT22, JP3 to LNODEMCU, JP4 to RNODEMCU, JP5 to GROVE
Changed lines of the file:
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@@
 </autorouter>
 <elements>
-<element name="JP1" library="pinhead" library_urn="urn:adsk.eagle:library:325" package="1X04" package3d_urn="urn:adsk.eagle:package:22407/2" value="" x="64.77" y="22.86" smashed="yes">
+<element name="SDS011" library="pinhead" library_urn="urn:adsk.eagle:library:325" package="1X04" package3d_urn="urn:adsk.eagle:package:22407/2" value="" x="64.77" y="22.86" smashed="yes">
 <attribute name="NAME" x="59.6138" y="24.6888" size="1.27" layer="25" ratio="10"/>
 <attribute name="POPULARITY" value="91" x="83.82" y="7.62" size="1.778" layer="27" display="off"/>
 <attribute name="VALUE" x="59.69" y="19.685" size="1.27" layer="27"/>
 </element>
-<element name="JP2" library="pinhead" library_urn="urn:adsk.eagle:library:325" package="1X03" package3d_urn="urn:adsk.eagle:package:22458/2" value="" x="76.2" y="50.8" smashed="yes" rot="R270">
+<element name="DHT22" library="pinhead" library_urn="urn:adsk.eagle:library:325" package="1X03" package3d_urn="urn:adsk.eagle:package:22458/2" value="" x="76.2" y="50.8" smashed="yes" rot="R270">
 <attribute name="NAME" x="78.0288" y="54.6862" size="1.27" layer="25" ratio="10" rot="R270"/>
 <attribute name="POPULARITY" value="92" x="60.96" y="21.59" size="1.778" layer="27" rot="R270" display="off"/>
 <attribute name="VALUE" x="73.025" y="54.61" size="1.27" layer="27" rot="R270"/>
 </element>
-<element name="JP3" library="pinhead" library_urn="urn:adsk.eagle:library:325" package="1X15" package3d_urn="urn:adsk.eagle:package:22424/2" value="" x="24.13" y="49.53" smashed="yes" rot="R270">
+<element name="LNODEMCU" library="pinhead" library_urn="urn:adsk.eagle:library:325" package="1X15" package3d_urn="urn:adsk.eagle:package:22424/2" value="" x="24.13" y="49.53" smashed="yes" rot="R270">
 <attribute name="NAME" x="25.9588" y="68.6562" size="1.27" layer="25" ratio="10" rot="R270"/>
 <attribute name="POPULARITY" value="4" x="21.59" y="16.51" size="1.778" layer="27" rot="R270" display="off"/>
 <attribute name="VALUE" x="20.955" y="68.58" size="1.27" layer="27" rot="R270"/>
 </element>
-<element name="JP4" library="pinhead" library_urn="urn:adsk.eagle:library:325" package="1X15" package3d_urn="urn:adsk.eagle:package:22424/2" value="" x="46.99" y="49.53" smashed="yes" rot="R270">
+<element name="RNODEMCU" library="pinhead" library_urn="urn:adsk.eagle:library:325" package="1X15" package3d_urn="urn:adsk.eagle:package:22424/2" value="" x="46.99" y="49.53" smashed="yes" rot="R270">
 <attribute name="NAME" x="48.8188" y="68.6562" size="1.27" layer="25" ratio="10" rot="R270"/>
 <attribute name="POPULARITY" value="4" x="38.1" y="16.51" size="1.778" layer="27" rot="R270" display="off"/>
 <attribute name="VALUE" x="43.815" y="68.58" size="1.27" layer="27" rot="R270"/>
 </element>
-<element name="JP5" library="pinhead" package="1X04M" value="" x="68.58" y="73.66" smashed="yes">
+<element name="GROVE" library="pinhead" package="1X04M" value="" x="68.58" y="73.66" smashed="yes">
 <attribute name="NAME" x="63.58" y="72.66" size="1.016" layer="25" ratio="14" rot="R90"/>
 <attribute name="VALUE" x="74.58" y="72.66" size="0.8128" layer="27" ratio="10" rot="R90"/>
@@
 <signals>
 <signal name="N$1">
-<contactref element="JP4" pad="2"/>
-<contactref element="JP5" pad="1"/>
+<contactref element="RNODEMCU" pad="2"/>
+<contactref element="GROVE" pad="1"/>
 <wire x1="56.515" y1="64.77" x2="65.405" y2="73.66" width="0.3048" layer="1"/>
 <wire x1="46.99" y1="64.77" x2="56.515" y2="64.77" width="0.3048" layer="1"/>
@@
 </signal>
 <signal name="N$2">
-<contactref element="JP4" pad="3"/>
-<contactref element="JP5" pad="2"/>
+<contactref element="RNODEMCU" pad="3"/>
+<contactref element="GROVE" pad="2"/>
 <wire x1="67.31" y1="73.66" x2="67.58" y2="73.66" width="0.3048" layer="1"/>
 <wire x1="46.99" y1="62.23" x2="63.5" y2="62.23" width="0.3048" layer="1"/>
@@
 </signal>
 <signal name="N$3">
-<contactref element="JP4" pad="5"/>
-<contactref element="JP1" pad="4"/>
+<contactref element="RNODEMCU" pad="5"/>
+<contactref element="SDS011" pad="4"/>
 <wire x1="66.04" y1="57.15" x2="68.58" y2="54.61" width="0.3048" layer="16"/>
 <wire x1="68.58" y1="54.61" x2="68.58" y2="22.86" width="0.3048" layer="16"/>
@@
 </signal>
 <signal name="N$4">
-<contactref element="JP4" pad="8"/>
-<contactref element="JP2" pad="2"/>
+<contactref element="RNODEMCU" pad="8"/>
+<contactref element="DHT22" pad="2"/>
 <wire x1="48.26" y1="50.8" x2="46.99" y2="49.53" width="0.3048" layer="1"/>
 <wire x1="76.2" y1="50.8" x2="48.26" y2="50.8" width="0.3048" layer="1"/>
 </signal>
 <signal name="N$5">
-<contactref element="JP4" pad="9"/>
-<contactref element="JP1" pad="3"/>
+<contactref element="RNODEMCU" pad="9"/>
+<contactref element="SDS011" pad="3"/>
 <wire x1="49.2125" y1="39.6875" x2="66.04" y2="22.86" width="0.3048" layer="16"/>
 <wire x1="49.2125" y1="44.7675" x2="49.2125" y2="39.6875" width="0.3048" layer="16"/>
@@
 </signal>
 <signal name="N$6">
-<contactref element="JP3" pad="15"/>
-<contactref element="JP1" pad="1"/>
-<contactref element="JP2" pad="1"/>
-<contactref element="JP5" pad="3"/>
+<contactref element="LNODEMCU" pad="15"/>
+<contactref element="SDS011" pad="1"/>
+<contactref element="DHT22" pad="1"/>
+<contactref element="GROVE" pad="3"/>
 <wire x1="69.85" y1="73.66" x2="69.58" y2="73.66" width="0.3048" layer="1"/>
 <wire x1="33.02" y1="22.86" x2="24.13" y2="31.75" width="0.3048" layer="1"/>
@@
 </signal>
 <signal name="N$7">
-<contactref element="JP3" pad="14"/>
-<contactref element="JP5" pad="4"/>
-<contactref element="JP2" pad="3"/>
-<contactref element="JP1" pad="2"/>
+<contactref element="LNODEMCU" pad="14"/>
+<contactref element="GROVE" pad="4"/>
+<contactref element="DHT22" pad="3"/>
+<contactref element="SDS011" pad="2"/>
 <wire x1="73.9775" y1="71.4375" x2="71.755" y2="73.66" width="0.3048" layer="16"/>
 <wire x1="73.9775" y1="50.4825" x2="73.9775" y2="71.4375" width="0.3048" layer="16"/>

Commit message: Modify Board
Parts:
- moved SDS011 28.4 mm to (36.8, 17.8), turned to 90 degrees
Routing:
- net N$7: track 100.9 -> 202.7 mm
- net N$6: track 113.8 -> 146.5 mm
- net N$5: track 32.0 -> 55.9 mm
- net N$3: track 54.4 -> 42.7 mm
- net N$2: track 29.8 -> 25.4 mm
Changed lines of the file:
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@@
 </variantdefs>
 <classes>
-<class number="0" name="default" width="0.3048" drill="0.508">
+<class number="0" name="default" width="0.508" drill="0.3048">
 <clearance class="0" value="0.254"/>
 </class>
@@
 </autorouter>
 <elements>
-<element name="SDS011" library="pinhead" library_urn="urn:adsk.eagle:library:325" package="1X04" package3d_urn="urn:adsk.eagle:package:22407/2" value="" x="64.77" y="22.86" smashed="yes">
-<attribute name="NAME" x="59.6138" y="24.6888" size="1.27" layer="25" ratio="10"/>
-<attribute name="POPULARITY" value="91" x="83.82" y="7.62" size="1.778" layer="27" display="off"/>
-<attribute name="VALUE" x="59.69" y="19.685" size="1.27" layer="27"/>
+<element name="SDS011" library="pinhead" library_urn="urn:adsk.eagle:library:325" package="1X04" package3d_urn="urn:adsk.eagle:package:22407/2" value="" x="36.83" y="17.78" smashed="yes" rot="R90">
+<attribute name="NAME" x="35.0012" y="12.6238" size="1.27" layer="25" ratio="10" rot="R90"/>
+<attribute name="POPULARITY" value="91" x="52.07" y="36.83" size="1.778" layer="27" rot="R90" display="off"/>
+<attribute name="VALUE" x="40.005" y="12.7" size="1.27" layer="27" rot="R90"/>
 </element>
 <element name="DHT22" library="pinhead" library_urn="urn:adsk.eagle:library:325" package="1X03" package3d_urn="urn:adsk.eagle:package:22458/2" value="" x="76.2" y="50.8" smashed="yes" rot="R270">
@@
 <contactref element="RNODEMCU" pad="2"/>
 <contactref element="GROVE" pad="1"/>
-<wire x1="56.515" y1="64.77" x2="65.405" y2="73.66" width="0.3048" layer="1"/>
-<wire x1="46.99" y1="64.77" x2="56.515" y2="64.77" width="0.3048" layer="1"/>
-<wire x1="65.405" y1="73.66" x2="65.58" y2="73.66" width="0.3048" layer="1"/>
+<wire x1="46.99" y1="64.77" x2="48.26" y2="66.04" width="0.508" layer="1"/>
+<wire x1="48.26" y1="66.04" x2="48.27805625" y2="66.04" width="0.508" layer="1"/>
+<wire x1="55.89805625" y1="73.66" x2="65.58" y2="73.66" width="0.508" layer="1"/>
+<wire x1="48.27805625" y1="66.04" x2="55.89805625" y2="73.66" width="0.508" layer="1"/>
 </signal>
 <signal name="N$2">
 <contactref element="RNODEMCU" pad="3"/>
 <contactref element="GROVE" pad="2"/>
-<wire x1="67.31" y1="73.66" x2="67.58" y2="73.66" width="0.3048" layer="1"/>
-<wire x1="46.99" y1="62.23" x2="63.5" y2="62.23" width="0.3048" layer="1"/>
-<wire x1="63.5" y1="62.23" x2="67.31" y2="66.04" width="0.3048" layer="1"/>
-<wire x1="67.31" y1="66.04" x2="67.31" y2="73.66" width="0.3048" layer="1"/>
+<wire x1="46.99" y1="62.23" x2="48.26" y2="63.5" width="0.508" layer="1"/>
+<wire x1="66.7992" y1="72.73838125" x2="66.7992" y2="72.8792" width="0.508" layer="1"/>
+<wire x1="66.7992" y1="72.8792" x2="67.58" y2="73.66" width="0.508" layer="1"/>
+<wire x1="48.26" y1="63.5" x2="57.56081875" y2="63.5" width="0.508" layer="1"/>
+<wire x1="57.56081875" y1="63.5" x2="66.7992" y2="72.73838125" width="0.508" layer="1"/>
 </signal>
 <signal name="N$3">
 <contactref element="RNODEMCU" pad="5"/>
 <contactref element="SDS011" pad="4"/>
-<wire x1="66.04" y1="57.15" x2="68.58" y2="54.61" width="0.3048" layer="16"/>
-<wire x1="68.58" y1="54.61" x2="68.58" y2="22.86" width="0.3048" layer="16"/>
-<wire x1="46.99" y1="57.15" x2="66.04" y2="57.15" width="0.3048" layer="16"/>
+<wire x1="36.83" y1="21.59" x2="36.83" y2="52.07" width="0.508" layer="1"/>
+<wire x1="36.83" y1="52.07" x2="41.91" y2="57.15" width="0.508" layer="1"/>
+<wire x1="41.91" y1="57.15" x2="46.99" y2="57.15" width="0.508" layer="1"/>
 </signal>
 <signal name="N$4">
 <contactref element="RNODEMCU" pad="8"/>
 <contactref element="DHT22" pad="2"/>
-<wire x1="48.26" y1="50.8" x2="46.99" y2="49.53" width="0.3048" layer="1"/>
-<wire x1="76.2" y1="50.8" x2="48.26" y2="50.8" width="0.3048" layer="1"/>
+<wire x1="46.99" y1="49.53" x2="74.93" y2="49.53" width="0.508" layer="1"/>
+<wire x1="74.93" y1="49.53" x2="76.2" y2="50.8" width="0.508" layer="1"/>
 </signal>
 <signal name="N$5">
 <contactref element="RNODEMCU" pad="9"/>
 <contactref element="SDS011" pad="3"/>
-<wire x1="49.2125" y1="39.6875" x2="66.04" y2="22.86" width="0.3048" layer="16"/>
-<wire x1="49.2125" y1="44.7675" x2="49.2125" y2="39.6875" width="0.3048" layer="16"/>
-<wire x1="46.99" y1="46.99" x2="49.2125" y2="44.7675" width="0.3048" layer="16"/>
+<wire x1="36.83" y1="19.05" x2="55.88" y2="19.05" width="0.508" layer="1"/>
+<wire x1="55.88" y1="19.05" x2="62.23" y2="25.4" width="0.508" layer="1"/>
+<wire x1="48.27805625" y1="45.72" x2="48.26" y2="45.72" width="0.508" layer="1"/>
+<wire x1="48.26" y1="45.72" x2="46.99" y2="46.99" width="0.508" layer="1"/>
+<wire x1="62.23" y1="25.4" x2="62.23" y2="31.76805625" width="0.508" layer="1"/>
+<wire x1="62.23" y1="31.76805625" x2="48.27805625" y2="45.72" width="0.508" layer="1"/>
 </signal>
 <signal name="N$6">
@@
 <contactref element="DHT22" pad="1"/>
 <contactref element="GROVE" pad="3"/>
-<wire x1="69.85" y1="73.66" x2="69.58" y2="73.66" width="0.3048" layer="1"/>
-<wire x1="33.02" y1="22.86" x2="24.13" y2="31.75" width="0.3048" layer="1"/>
-<wire x1="60.96" y1="22.86" x2="33.02" y2="22.86" width="0.3048" layer="1"/>
-<wire x1="78.4225" y1="51.1175" x2="76.2" y2="53.34" width="0.3048" layer="16"/>
-<wire x1="78.4225" y1="30.1625" x2="78.4225" y2="51.1175" width="0.3048" layer="16"/>
-<wire x1="68.8975" y1="20.6375" x2="78.4225" y2="30.1625" width="0.3048" layer="16"/>
-<wire x1="60.96" y1="20.6375" x2="68.8975" y2="20.6375" width="0.3048" layer="16"/>
-<wire x1="60.96" y1="22.86" x2="60.96" y2="20.6375" width="0.3048" layer="16"/>
-<wire x1="69.58" y1="73.66" x2="69.85" y2="73.39" width="0.3048" layer="1"/>
-<wire x1="69.85" y1="55.88" x2="72.39" y2="53.34" width="0.3048" layer="1"/>
-<wire x1="72.39" y1="53.34" x2="76.2" y2="53.34" width="0.3048" layer="1"/>
-<wire x1="69.85" y1="73.39" x2="69.85" y2="55.88" width="0.3048" layer="1"/>
+<wire x1="24.13" y1="31.75" x2="25.4" y2="30.48" width="0.508" layer="1"/>
+<wire x1="25.4" y1="30.48" x2="25.4" y2="13.97" width="0.508" layer="1"/>
+<wire x1="25.4" y1="13.97" x2="36.83" y2="13.97" width="0.508" layer="1"/>
+<wire x1="36.83" y1="13.97" x2="72.39" y2="13.97" width="0.508" layer="1"/>
+<wire x1="72.39" y1="13.97" x2="88.9" y2="30.48" width="0.508" layer="1"/>
+<wire x1="88.9" y1="30.48" x2="88.9" y2="52.07" width="0.508" layer="1"/>
+<wire x1="88.9" y1="52.07" x2="87.63" y2="53.34" width="0.508" layer="1"/>
+<wire x1="87.63" y1="53.34" x2="76.2" y2="53.34" width="0.508" layer="1"/>
+<wire x1="69.58" y1="73.66" x2="76.2" y2="67.04" width="0.508" layer="1"/>
+<wire x1="76.2" y1="67.04" x2="76.2" y2="53.34" width="0.508" layer="1"/>
 </signal>
 <signal name="N$7">
@@
 <contactref element="DHT22" pad="3"/>
 <contactref element="SDS011" pad="2"/>
-<wire x1="73.9775" y1="71.4375" x2="71.755" y2="73.66" width="0.3048" layer="16"/>
-<wire x1="73.9775" y1="50.4825" x2="73.9775" y2="71.4375" width="0.3048" layer="16"/>
-<wire x1="76.2" y1="48.26" x2="73.9775" y2="50.4825" width="0.3048" layer="16"/>
-<wire x1="71.755" y1="73.66" x2="71.58" y2="73.66" width="0.3048" layer="16"/>
-<wire x1="33.3375" y1="25.0825" x2="24.13" y2="34.29" width="0.3048" layer="1"/>
-<wire x1="61.2775" y1="25.0825" x2="33.3375" y2="25.0825" width="0.3048" layer="1"/>
-<wire x1="63.5" y1="22.86" x2="61.2775" y2="25.0825" width="0.3048" layer="1"/>
-<wire x1="61.2775" y1="33.3375" x2="76.2" y2="48.26" width="0.3048" layer="1"/>
-<wire x1="61.2775" y1="25.0825" x2="61.2775" y2="33.3375" width="0.3048" layer="1"/>
+<wire x1="24.13" y1="34.29" x2="27.94" y2="34.29" width="0.508" layer="1"/>
+<wire x1="30.48" y1="31.75" x2="30.48" y2="16.51" width="0.508" layer="1"/>
+<wire x1="30.48" y1="16.51" x2="31.75" y2="15.24" width="0.508" layer="1"/>
+<wire x1="31.75" y1="15.24" x2="36.83" y2="15.24" width="0.508" layer="1"/>
+<wire x1="36.83" y1="15.24" x2="36.83" y2="16.51" width="0.508" layer="1"/>
+<wire x1="27.94" y1="34.29" x2="30.48" y2="31.75" width="0.508" layer="1"/>
+<wire x1="36.83" y1="16.51" x2="63.5" y2="16.51" width="0.508" layer="1"/>
+<wire x1="76.2" y1="29.21" x2="76.2" y2="48.26" width="0.508" layer="1"/>
+<wire x1="63.5" y1="16.51" x2="76.2" y2="29.21" width="0.508" layer="1"/>
+<wire x1="36.83" y1="16.51" x2="34.29" y2="16.51" width="0.508" layer="1"/>
+<wire x1="34.29" y1="16.51" x2="33.02" y2="17.78" width="0.508" layer="1"/>
+<wire x1="33.02" y1="17.78" x2="33.02" y2="76.2" width="0.508" layer="1"/>
+<wire x1="33.02" y1="76.2" x2="38.1" y2="81.28" width="0.508" layer="1"/>
+<wire x1="38.1" y1="81.28" x2="64.77" y2="81.28" width="0.508" layer="1"/>
+<wire x1="64.77" y1="81.28" x2="72.39" y2="73.66" width="0.508" layer="1"/>
+<wire x1="72.39" y1="73.66" x2="71.58" y2="73.66" width="0.508" layer="1"/>
 </signal>
 </signals>
