File: EagleAirPoll/SchemaFin.sch (EAGLE design)
At the start: 5 parts

Commit message: Remove consistency errors
Parts:
- DHT22: value Temp&Humidity -> (none)
- GROVE: value Gases sensor -> (none)
- SDS011: value Dust Sensor -> (none)
Changed lines of the file:
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@@
 </classes>
 <parts>
-<part name="SDS011" library="pinhead" library_urn="urn:adsk.eagle:library:325" deviceset="PINHD-1X4" device="" package3d_urn="urn:adsk.eagle:package:22407/2" value="Dust Sensor"/>
-<part name="DHT22" library="pinhead" library_urn="urn:adsk.eagle:library:325" deviceset="PINHD-1X3" device="" package3d_urn="urn:adsk.eagle:package:22458/2" value="Temp&amp;Humidity"/>
+<part name="SDS011" library="pinhead" library_urn="urn:adsk.eagle:library:325" deviceset="PINHD-1X4" device="" package3d_urn="urn:adsk.eagle:package:22407/2"/>
+<part name="DHT22" library="pinhead" library_urn="urn:adsk.eagle:library:325" deviceset="PINHD-1X3" device="" package3d_urn="urn:adsk.eagle:package:22458/2"/>
 <part name="LNODEMCU" library="pinhead" library_urn="urn:adsk.eagle:library:325" deviceset="PINHD-1X15" device="" package3d_urn="urn:adsk.eagle:package:22424/2"/>
 <part name="RNODEMCU" library="pinhead" library_urn="urn:adsk.eagle:library:325" deviceset="PINHD-1X15" device="" package3d_urn="urn:adsk.eagle:package:22424/2"/>
-<part name="GROVE" library="pinhead" deviceset="PINHD-1X4" device="M" value="Gases sensor"/>
+<part name="GROVE" library="pinhead" deviceset="PINHD-1X4" device="M"/>
 </parts>
 <sheets>
